File: PCB/Multilevel_Schmitt.sch (KiCad schematic (older format))
At the start: 24 parts, among them J1 Conn_02x03_Counter_Clockwise, J2 Conn_01x03, J3 Conn_01x08_Female, J4 Conn_01x08_Female, J5 Conn_01x02, Q1 BS170, U1 ATtiny84-20PU, U2 74HC14, U3 MCP1700-2502E_TO92, U4 74HC4051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

Commit message: last changes to master
Parts:
- removed D1: D, Diode_THT:D_DO-15_P10.16mm_Horizontal, symbol Device:D
- added D1: 1N5817, Diode_THT:D_DO-41_SOD81_P10.16mm_Horizontal, symbol Diode:1N5817
Connections:
- net at C5.1, U3.2 (VI): now also D1.1 (K)
- net at J2.2 (Pin_2), J5.2 (Pin_2): now also D1.2 (A)
Changed lines of the file:
@@
 	4250 5650 4400 5650
-$Comp
-L Device:D D1
-U 1 1 6055F6A7
-P 4500 6150
-F 0 "D1" H 4500 6300 50  0000 C CNN
-F 1 "D" H 4500 6000 50  0000 C CNN
-F 2 "Diode_THT:D_DO-15_P10.16mm_Horizontal" H 4500 6150 50  0001 C CNN
-F 3 "~" H 4500 6150 50  0001 C CNN
-	1    4500 6150
-	-1   0    0    1
-$EndComp
 $Comp
 L Device:R R1
@@
 	-1   0    0    1
 $EndComp
+$Comp
+L Diode:1N5817 D1
+U 1 1 60810178
+P 4500 6150
+F 0 "D1" H 4500 5933 50  0000 C CNN
+F 1 "1N5817" H 4500 6024 50  0000 C CNN
+F 2 "Diode_THT:D_DO-41_SOD81_P10.16mm_Horizontal" H 4500 5975 50  0001 C CNN
+F 3 "http://www.vishay.com/docs/88525/1n5817.pdf" H 4500 6150 50  0001 C CNN
+	1    4500 6150
+	-1   0    0    1
+$EndComp
