File: PCB/Multilevel_Schmitt.kicad_pcb (KiCad board)
At the start: 2 copper layers, 32 x 102 mm, 24 parts, among them J1 Conn_02x03_Counter_Clockwise, J2 Conn_01x03, J3 Conn_01x08_Female, J4 Conn_01x08_Female, J5 Conn_01x02, Q1 BS170, U1 ATtiny84-20PU, U2 74HC14, U3 MCP1700-2502E_TO92, U4 74HC4051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

Commit message: last changes to master
Parts:
- moved J2 0.50 mm to (103.5, 49.0)
- moved J5 0.50 mm to (112.5, 49.0)
- moved J1 0.42 mm to (128.5, 54.1)
Routing:
- net SCL_SCK: track 50.7 -> 54.4 mm
- net M0: track 251.9 -> 255.2 mm
- net POW_TX: track 17.5 -> 18.8 mm
- net Net-(D1-Pad2): track 17.2 -> 18.2 mm
- net SDA_MOSI: track 54.2 -> 54.8 mm
